File: kicad/Phase and Filter/phase v3.kicad_pcb (KiCad board)
At the start: 2 copper layers, 80 x 51 mm, 51 parts, among them J1 AUDIO_JACK_3.5MM_KIT, J2 AUDIO_JACK_3.5MM_KIT, J3 Pad, J4 Pad, U1 LM358DIP08-SOIC, U2 LM358, U3 LM358, U4 LM358DIP08-SOIC

Commit message: fix kicad
Parts:
- J1, J2: footprint phase v3:AUDIO-JACK-KIT -> Xenir:Audio_Jack
- VR1: value 50k -> Trimpot; footprint phase v3:TRIMPOT-PTH-3386U -> Xenir:Trimpot
- VR2: value 500k -> Trimpot; footprint phase v3:TRIMPOT-PTH-3386U -> Xenir:Trimpot
- VR3: value 500 -> Trimpot; footprint phase v3:TRIMPOT-PTH-3386U -> Xenir:Trimpot
- moved J2 8.79 mm to (142.2, 111.8)
- moved J1 8.55 mm to (81.0, 106.0)
- moved VR3 5.27 mm to (123.8, 121.0), turned to 270 degrees
- moved VR1 5.02 mm to (99.0, 103.5), turned to 270 degrees
- moved VR2 5.00 mm to (117.2, 103.8), turned to 270 degrees
Connections:
- VR1 pad 1: Net-(C4-Pad1) -> Net-(J1-PadRING)
- VR1 pad 3: Net-(J1-PadRING) -> Net-(C4-Pad1)
- VR2 pad 1: Net-(C2-Pad1) -> Net-(R3-Pad2)
- VR2 pad 3: Net-(R3-Pad2) -> Net-(C2-Pad1)
- VR3 pad 1: Net-(R10-Pad1) -> Net-(R13-Pad2)
- VR3 pad 3: Net-(R13-Pad2) -> Net-(R10-Pad1)
