File: kicad/Mixer-ADE/Mixer-ADE.sch (KiCad schematic (older format))
At the start: 32 parts, among them J1 Audio_Jack, J2 BNC, J3 BNC, J6 BNC, M1 ADEX-10L, M2 ADEX-10L, T3 T37_XFRM

Commit message: replace T
Parts:
- removed T3: T37_XFRM, Xenir:T37 Transformer, symbol Xenir:T37_XFRM
- added T1: T50_SPLITTER, Xenir:T50 Trifilar, symbol Xenir:T50_SPLITTER
Connections:
- wire segments 52 -> 45
Other:
- moved on the sheet: J6
Changed lines of the file:
@@
 	2050 1400 2050 1500
-$Comp
-L Xenir:T37_XFRM T3
-U 1 1 5EC79379
-P 8850 3300
-F 0 "T3" H 8850 2450 50  0000 C CNN
-F 1 "T37_XFRM" H 8850 3300 50  0000 C CNN
-F 2 "Xenir:T37 Transformer" H 8850 3300 50  0001 C CNN
-F 3 "" H 8850 3300 50  0001 C CNN
-	1    8850 3300
-	1    0    0    -1
-$EndComp
-$Comp
-L Xenir:Resistor R5
-U 1 1 5EC79D0C
-P 8100 3750
-F 0 "R5" H 8100 3825 28  0000 C CNN
-F 1 "100" H 8100 3675 28  0000 C CNN
-F 2 "Resistor_THT:R_Axial_DIN0204_L3.6mm_D1.6mm_P2.54mm_Vertical" H 8100 3650 50  0001 C CNN
-F 3 "" H 8100 3650 50  0001 C CNN
-	1    8100 3750
-	0    -1   -1   0
-$EndComp
-Wire Wire Line
-	8100 3950 8100 4050
-Wire Wire Line
-	9250 3250 9250 3450
-Wire Wire Line
-	8100 3550 8100 3250
-Wire Wire Line
-	8450 3450 8350 3450
-Wire Wire Line
-	8350 3450 8350 4250
-Wire Wire Line
-	8350 4250 9250 4250
-Wire Wire Line
-	9250 4250 9250 4050
 $Comp
 L power:GND #PWR0118
 U 1 1 5EC88413
-P 9950 4250
-F 0 "#PWR0118" H 9950 4000 50  0001 C CNN
-F 1 "GND" H 9950 4100 50  0000 C CNN
-F 2 "" H 9950 4250 50  0001 C CNN
-F 3 "" H 9950 4250 50  0001 C CNN
-	1    9950 4250
+P 9200 3500
+F 0 "#PWR0118" H 9200 3250 50  0001 C CNN
+F 1 "GND" H 9200 3350 50  0000 C CNN
+F 2 "" H 9200 3500 50  0001 C CNN
+F 3 "" H 9200 3500 50  0001 C CNN
+	1    9200 3500
 	1    0    0    -1
 $EndComp
@@
 L Xenir:BNC J6
 U 1 1 5EC8841E
-P 9950 4050
-F 0 "J6" H 9850 3900 50  0000 C CNN
-F 1 "BNC" H 9950 4200 50  0000 C CNN
-F 2 "Xenir:BNC" H 9950 4200 50  0001 C CNN
-F 3 "" H 9950 4200 50  0001 C CNN
-	1    9950 4050
+P 9200 3300
+F 0 "J6" H 9100 3150 50  0000 C CNN
+F 1 "BNC" H 9200 3450 50  0000 C CNN
+F 2 "Xenir:BNC" H 9200 3450 50  0001 C CNN
+F 3 "" H 9200 3450 50  0001 C CNN
+	1    9200 3300
 	-1   0    0    -1
 $EndComp
-Wire Wire Line
-	9250 4050 9750 4050
-Connection ~ 9250 4050
-Wire Wire Line
-	8100 4050 8450 4050
-Wire Wire Line
-	8100 3250 9250 3250
 $Comp
 L power:GND #PWR0101
@@
 	4450 2750 8100 2750
 Wire Wire Line
-	8100 2750 8100 3250
-Connection ~ 8100 3250
-Wire Wire Line
 	8100 4500 4450 4500
 Wire Wire Line
 	4450 4500 4450 4000
-Wire Wire Line
-	8100 4050 8100 4500
-Connection ~ 8100 4050
+$Comp
+L Xenir:T50_SPLITTER T1
+U 1 1 5ECADD18
+P 8450 4300
+F 0 "T1" H 8450 3050 50  0000 C CNN
+F 1 "T50_SPLITTER" H 8450 4200 50  0000 C CNN
+F 2 "Xenir:T50 Trifilar" H 8450 4300 50  0001 C CNN
+F 3 "" H 8450 4300 50  0001 C CNN
+	1    8450 4300
+	-1   0    0    1
+$EndComp
+$Comp
+L Xenir:Resistor R5
+U 1 1 5ECB02BC
+P 7800 3700
+F 0 "R5" H 7800 3775 28  0000 C CNN
+F 1 "100" H 7800 3625 28  0000 C CNN
+F 2 "Resistor_THT:R_Axial_DIN0204_L3.6mm_D1.6mm_P2.54mm_Vertical" H 7800 3600 50  0001 C CNN
+F 3 "" H 7800 3600 50  0001 C CNN
+	1    7800 3700
+	0    -1   -1   0
+$EndComp
+$Comp
+L power:GND #PWR0119
+U 1 1 5ECB190D
+P 7800 3900
+F 0 "#PWR0119" H 7800 3650 50  0001 C CNN
+F 1 "GND" H 7800 3750 50  0000 C CNN
+F 2 "" H 7800 3900 50  0001 C CNN
+F 3 "" H 7800 3900 50  0001 C CNN
+	1    7800 3900
+	1    0    0    -1
+$EndComp
+Wire Wire Line
+	8100 3500 7800 3500
+Wire Wire Line
+	8100 3700 8100 3500
+Connection ~ 8100 3500
+Wire Wire Line
+	8100 2750 8100 3100
+Wire Wire Line
+	8100 4100 8100 4500
+Wire Wire Line
+	8800 3300 9000 3300
+$Comp
+L power:GND #PWR0120
+U 1 1 5ECBBC48
+P 8800 3900
+F 0 "#PWR0120" H 8800 3650 50  0001 C CNN
+F 1 "GND" H 8800 3750 50  0000 C CNN
+F 2 "" H 8800 3900 50  0001 C CNN
+F 3 "" H 8800 3900 50  0001 C CNN
+	1    8800 3900
+	1    0    0    -1
+$EndComp
 $EndSCHEMATC

Commit message: Update Mixer-ADE.sch
Parts:
- T1: value T50_SPLITTER -> FT50-43 Trifilar
Changed lines of the file:
@@
 P 8450 4300
 F 0 "T1" H 8450 3050 50  0000 C CNN
-F 1 "T50_SPLITTER" H 8450 4200 50  0000 C CNN
+F 1 "FT50-43 Trifilar" H 8450 4200 50  0000 C CNN
 F 2 "Xenir:T50 Trifilar" H 8450 4300 50  0001 C CNN
 F 3 "" H 8450 4300 50  0001 C CNN
