File: kicad/Microphone Amp/Microphone Amp.kicad_pcb (KiCad board)
At the start: 2 copper layers, 73.5 x 48 mm, 24 parts, among them J1 Pad, J2 Pad, J4 Audio_Jack, M1 Electret, U3 LM358

Commit message: u
Parts:
- C4: value .1uF -> 1uF
- R7: value 4.7k -> 20k
Changed lines of the file:
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@@
       (effects (font (size 0.5 0.5) (thickness 0.125)))
     )
-    (fp_text value 4.7k (at 0 1) (layer F.Fab)
+    (fp_text value 20k (at 0 1) (layer F.Fab)
       (effects (font (size 0.5 0.5) (thickness 0.125)))
     )
@@
       (effects (font (size 0.5 0.5) (thickness 0.125)))
     )
-    (fp_text value .1uF (at 0.5 4 90) (layer F.Fab)
-      (effects (font (size 0.5 0.5) (thickness 0.125)))
-    )
+    (fp_text value 1uF (at 0.5 4 90) (layer F.Fab)
+      (effects (font (size 0.5 0.5) (thickness 0.125)))
+    )
