File: kicad/Microphone Amp/Microphone Amp.sch (KiCad schematic (older format))
At the start: 24 parts, among them J1 Pad, J2 Pad, J4 Audio_Jack, M1 Electret, U3 LM358

Commit message: u
Parts:
- C4: value .1uF -> 1uF
- R7: value 4.7k -> 20k
Changed lines of the file:
@@
 P 2400 3200
 F 0 "R7" H 2400 3275 28  0000 C CNN
-F 1 "4.7k" H 2400 3125 28  0000 C CNN
+F 1 "20k" H 2400 3125 28  0000 C CNN
 F 2 "Xenir:Resistor 0805" H 2400 3100 50  0001 C CNN
 F 3 "" H 2400 3100 50  0001 C CNN
@@
 P 5550 3550
 F 0 "C4" H 5550 3675 28  0000 C CNN
-F 1 ".1uF" H 5550 3425 28  0000 C CNN
+F 1 "1uF" H 5550 3425 28  0000 C CNN
 F 2 "Xenir:Capacitor 0805" H 5550 3400 50  0001 C CNN
 F 3 "" H 5550 3400 50  0001 C CNN

Commit message: u
Other:
- moved on the sheet: C1, C10, C2, C3, C4, C5, C6, C7, J1, J2, J4, L1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
